File: IN-12Panel.kicad_pcb (KiCad board)
At the start: 2 copper layers, 84 x 50 mm, 12 parts, among them J1 Conn_01x04_Pin, J2 Conn_01x04_Pin, J3 Conn_01x11_Pin, J4 Conn_01x11_Pin, U1 IN-12, U2 IN-12, U3 IN-12, U4 IN-12

Commit message: 基板結合にあたり，コネクタの位置・向きを変更
Parts:
- J3, J4: value Conn_01x11_Pin -> Conn_01x12_Pin; footprint Connector_JST:JST_XH_S11B-XH-A_1x11_P2.50mm_Horizontal -> Connector_JST:JST_XH_S12B-XH-A_1x12_P2.50mm_Horizontal
- moved J1 42.0 mm to (17.2, 9.50)
- moved J3 20.3 mm to (39.2, 9.50)
- moved J4 0.75 mm to (44.8, 40.5)
Routing:
- net /1: track 0.00 -> 120.2 mm, vias 0 -> 2
- net /DIG0: track 0.00 -> 119.5 mm
- net /7: track 0.00 -> 117.7 mm, vias 0 -> 2
- net /9: track 0.00 -> 116.3 mm, vias 0 -> 1
- net /3: track 0.00 -> 115.7 mm, vias 0 -> 2
- net /2: track 0.00 -> 115.1 mm, vias 0 -> 2
- net /LHDP: track 0.00 -> 114.6 mm, vias 0 -> 2
- net /0: track 0.00 -> 114.5 mm, vias 0 -> 1
- net /5: track 0.00 -> 114.0 mm, vias 0 -> 2
- net /8: track 0.00 -> 113.7 mm, vias 0 -> 2
- net /4: track 0.00 -> 113.6 mm, vias 0 -> 2
- net /6: track 0.00 -> 113.3 mm, vias 0 -> 2
- net /DIG3: track 0.00 -> 107.1 mm
- net /DIG2: track 0.00 -> 75.5 mm
- net /DIG1: track 0.00 -> 74.8 mm

Commit message: 製造後データを追加
Other:
- board text added: "0"
- board text added: "1"
- board text added: "2"
- board text added: "3"
- board text added: "4"
- board text added: "5"
- board text added: "6"
- board text added: "7"
- board text added: "8"
- board text added: "9"
- board text added: "DOT"
- board text added: "Digit Control"
- board text added: "JLCJLCJLCJLC"
- board text added: "NC"
- board text added: "Nixie Panel"
- board text added: "Value Control"
- board text added: "by T.N."
- board text added: "for IN-12"
